File: Dover Driver.sch (EAGLE design)
At the start: 44 parts

Commit message: Version 1.0 layout finished
Parts:
- added D1: LED3MM, mb_diodes:LED3MM
- added R16: 4k7, mb_resistors:6MM.3
- C10, C12, C3, C8: value 4k7 -> 4u7
- U$2: value MMBFj201 -> J201
- U$3, U$4, U$5: value MMBFJ201 -> J201
Connections:
- new net N$28: D1.A, R16.1
- new net N$29: D1.C, U$1.LED
- net N$5: now also R16.2
Other:
- moved on the sheet: C1
Changed lines of the file:
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@@
 <parts>
 <part name="U$1" library="xc_library" deviceset="BOARDLINK" device=""/>
-<part name="U$2" library="xc_library" deviceset="MMBF5458" device="" value="MMBFj201"/>
-<part name="U$3" library="xc_library" deviceset="MMBF5458" device="" value="MMBFJ201"/>
-<part name="U$4" library="xc_library" deviceset="MMBF5458" device="" value="MMBFJ201"/>
-<part name="U$5" library="xc_library" deviceset="MMBF5458" device="" value="MMBFJ201"/>
+<part name="U$2" library="xc_library" deviceset="MMBF5458" device="" value="J201"/>
+<part name="U$3" library="xc_library" deviceset="MMBF5458" device="" value="J201"/>
+<part name="U$4" library="xc_library" deviceset="MMBF5458" device="" value="J201"/>
+<part name="U$5" library="xc_library" deviceset="MMBF5458" device="" value="J201"/>
 <part name="R1" library="mb_resistors" deviceset="6MM" device=".3" value="1M"/>
 <part name="R2" library="mb_resistors" deviceset="6MM" device=".3" value="22K"/>
@@
 <part name="C1" library="mb_caps-electro" deviceset="063" device="1" value="100uF"/>
 <part name="C2" library="mb_caps-ceramic" deviceset="050X030_025" device="1" value="330pF"/>
-<part name="C3" library="mb_caps-electro" deviceset="050" device="1" value="4k7"/>
+<part name="C3" library="mb_caps-electro" deviceset="050" device="1" value="4u7"/>
 <part name="C4" library="mb_caps-chicklet" deviceset="075X040" device="2" value="100nF"/>
 <part name="C5" library="mb_caps-box" deviceset="072X025" device="2" value="47nF"/>
 <part name="C6" library="mb_caps-ceramic" deviceset="050X030_025" device="1" value="47pF"/>
 <part name="C7" library="mb_caps-ceramic" deviceset="050X030_025" device="1" value="330pF"/>
-<part name="C8" library="mb_caps-electro" deviceset="050" device="1" value="4k7"/>
+<part name="C8" library="mb_caps-electro" deviceset="050" device="1" value="4u7"/>
 <part name="C9" library="mb_caps-box" deviceset="072X025" device="2" value="10nF"/>
 <part name="GND11" library="mb_supply" deviceset="GND" device=""/>
-<part name="C10" library="mb_caps-electro" deviceset="050" device="1" value="4k7"/>
+<part name="C10" library="mb_caps-electro" deviceset="050" device="1" value="4u7"/>
 <part name="GND12" library="mb_supply" deviceset="GND" device=""/>
 <part name="GND13" library="mb_supply" deviceset="GND" device=""/>
 <part name="C11" library="mb_caps-box" deviceset="072X025" device="2" value="22nF"/>
 <part name="GND14" library="mb_supply" deviceset="GND" device=""/>
-<part name="C12" library="mb_caps-electro" deviceset="050" device="1" value="4k7"/>
+<part name="C12" library="mb_caps-electro" deviceset="050" device="1" value="4u7"/>
 <part name="GND15" library="mb_supply" deviceset="GND" device=""/>
 <part name="GND16" library="mb_supply" deviceset="GND" device=""/>
@@
 <part name="GND18" library="mb_supply" deviceset="GND" device=""/>
 <part name="GND19" library="mb_supply" deviceset="GND" device=""/>
+<part name="R16" library="mb_resistors" deviceset="6MM" device=".3" value="4k7"/>
+<part name="D1" library="mb_diodes" deviceset="LED" device="3MM"/>
 </parts>
 <sheets>
@@
 <instance part="U$2" gate="G$1" x="12.7" y="76.2" smashed="yes">
 <attribute name="NAME" x="9.144" y="70.612" size="1.778" layer="95"/>
-<attribute name="VALUE" x="13.716" y="81.28" size="1.778" layer="96" rot="R180"/>
+<attribute name="VALUE" x="18.796" y="77.47" size="1.778" layer="96" rot="R180"/>
 </instance>
 <instance part="U$3" gate="G$1" x="78.74" y="68.58" smashed="yes">
@@
 <attribute name="VALUE" x="0.635" y="84.455" size="1.778" layer="96" rot="R90"/>
 </instance>
-<instance part="GND3" gate="GND" x="10.414" y="85.598" smashed="yes">
-<attribute name="VALUE" x="8.509" y="82.423" size="1.778" layer="96"/>
+<instance part="GND3" gate="GND" x="10.414" y="83.566" smashed="yes">
+<attribute name="VALUE" x="8.509" y="80.391" size="1.778" layer="96"/>
 </instance>
 <instance part="GND4" gate="GND" x="15.24" y="50.8" smashed="yes">
@@
 <attribute name="VALUE" x="89.535" y="45.085" size="1.778" layer="96"/>
 </instance>
-<instance part="C1" gate="G$1" x="10.414" y="95.25" smashed="yes">
-<attribute name="NAME" x="11.43" y="95.885" size="1.778" layer="95"/>
-<attribute name="VALUE" x="12.573" y="89.154" size="1.778" layer="96" rot="R90"/>
+<instance part="C1" gate="G$1" x="10.414" y="93.218" smashed="yes">
+<attribute name="NAME" x="11.43" y="93.853" size="1.778" layer="95"/>
+<attribute name="VALUE" x="12.573" y="87.122" size="1.778" layer="96" rot="R90"/>
 </instance>
 <instance part="C2" gate="G$1" x="35.56" y="81.28" smashed="yes" rot="R90">
@@
 <instance part="GND19" gate="GND" x="218.44" y="63.5" smashed="yes">
 <attribute name="VALUE" x="216.535" y="60.325" size="1.778" layer="96"/>
+</instance>
+<instance part="R16" gate="G$1" x="5.08" y="88.9" smashed="yes" rot="R90">
+<attribute name="NAME" x="3.5814" y="87.249" size="1.778" layer="95" rot="R90"/>
+<attribute name="VALUE" x="7.112" y="82.55" size="1.778" layer="96" rot="R90"/>
+</instance>
+<instance part="D1" gate="G$1" x="-2.54" y="81.28" smashed="yes">
+<attribute name="NAME" x="-4.572" y="77.724" size="1.778" layer="95"/>
 </instance>
 </instances>
@@
 <pinref part="GND3" gate="GND" pin="GND"/>
 <pinref part="C1" gate="G$1" pin="-"/>
-<wire x1="10.414" y1="88.138" x2="10.414" y2="90.17" width="0.1524" layer="91"/>
+<wire x1="10.414" y1="86.106" x2="10.414" y2="88.138" width="0.1524" layer="91"/>
 </segment>
 <segment>
@@
 <wire x1="1.524" y1="83.82" x2="1.524" y2="99.06" width="0.1524" layer="91"/>
 <pinref part="TRIM1" gate="G$1" pin="3"/>
-<wire x1="1.524" y1="99.06" x2="10.414" y2="99.06" width="0.1524" layer="91"/>
-<pinref part="C1" gate="G$1" pin="+"/>
-<wire x1="10.414" y1="99.06" x2="15.24" y2="99.06" width="0.1524" layer="91"/>
-<wire x1="10.414" y1="97.79" x2="10.414" y2="99.06" width="0.1524" layer="91"/>
+<wire x1="1.524" y1="99.06" x2="5.08" y2="99.06" width="0.1524" layer="91"/>
+<wire x1="5.08" y1="99.06" x2="7.62" y2="99.06" width="0.1524" layer="91"/>
 <pinref part="TRIM2" gate="G$1" pin="3"/>
+<wire x1="7.62" y1="99.06" x2="15.24" y2="99.06" width="0.1524" layer="91"/>
 <wire x1="81.28" y1="99.06" x2="15.24" y2="99.06" width="0.1524" layer="91"/>
 <junction x="15.24" y="99.06"/>
@@
 <wire x1="167.64" y1="99.06" x2="124.46" y2="99.06" width="0.1524" layer="91"/>
 <junction x="124.46" y="99.06"/>
+<pinref part="R16" gate="G$1" pin="2"/>
+<wire x1="5.08" y1="93.98" x2="5.08" y2="99.06" width="0.1524" layer="91"/>
+<junction x="5.08" y="99.06"/>
+<pinref part="C1" gate="G$1" pin="+"/>
+<wire x1="10.414" y1="95.758" x2="7.62" y2="95.758" width="0.1524" layer="91"/>
+<wire x1="7.62" y1="95.758" x2="7.62" y2="99.06" width="0.1524" layer="91"/>
+<junction x="7.62" y="99.06"/>
 </segment>
 </net>
@@
 </segment>
 </net>
+<net name="N$28" class="0">
+<segment>
+<pinref part="R16" gate="G$1" pin="1"/>
+<pinref part="D1" gate="G$1" pin="A"/>
+<wire x1="5.08" y1="83.82" x2="5.08" y2="81.28" width="0.1524" layer="91"/>
+<wire x1="5.08" y1="81.28" x2="2.54" y2="81.28" width="0.1524" layer="91"/>
+</segment>
+</net>
+<net name="N$29" class="0">
+<segment>
+<pinref part="D1" gate="G$1" pin="C"/>
+<pinref part="U$1" gate="G$1" pin="LED"/>
+<wire x1="-5.08" y1="81.28" x2="-11.176" y2="81.28" width="0.1524" layer="91"/>
+</segment>
+</net>
